Commit message: Adjusted Monza_track.world

File: racecar_description/urdf/racecar.urdf.xacro (robot description, xacro)
@@ -37,8 +37,8 @@
   <!-- chassis_length is measured along the x axis, chassis_width
        along the y axis, and chassis_height along the z axis. -->
-  <xacro:property name="chassis_length" value="0.135"/>
-  <xacro:property name="chassis_width" value="0.36"/>
-  <xacro:property name="chassis_height" value="0.0021"/>
-  <xacro:property name="chassis_mass" value="1.26244"/>
+  <xacro:property name="chassis_length" value="0.258"/>
+  <xacro:property name="chassis_width" value="0.168"/>
+  <xacro:property name="chassis_height" value="0.01"/>
+  <xacro:property name="chassis_mass" value="2.788"/>
   <!-- battery_dist is the distance between the inner edges of the
        batteries. battery_comp_depth is the battery compartment depth.
@@ -49,8 +49,8 @@
   <xacro:property name="battery_comp_depth" value="0.02"/>
   <xacro:property name="battery_comp_angle" value="0.34906585"/>
-  <xacro:property name="battery_length" value="0.1"/>
-  <xacro:property name="battery_width" value="0.05"/>
-  <xacro:property name="battery_height" value="0.03"/>
-  <xacro:property name="battery_mass" value="0.05025"/>
+  <xacro:property name="battery_length" value="0.16"/>
+  <xacro:property name="battery_width" value="0.047"/>
+  <xacro:property name="battery_height" value="0.024"/>
+  <xacro:property name="battery_mass" value="0.5025"/>
   <!-- hub_dia and tire_dia are the diameters of the hub and tire,
        respectively. hex_hub_depth is the distance that the hex hub is

File: racecar_description/urdf/sensors/camera.xacro (robot description, xacro)
@@ -3,9 +3,9 @@
 	<link name="camera_link">
 	    <inertial>
-		<mass value="0.0052875" />
+		<mass value="0.001" />
 		<origin xyz="0 0 0" />
-		<inertia ixx="4.1e-07" ixy="0.0" ixz="0.0"
-		         iyy="7.9e-07" iyz="0.0"
-		         izz="4.1e-07" />
+		<inertia ixx="0.001" ixy="0.0" ixz="0.0"
+		         iyy="0.001" iyz="0.0"
+		         izz="0.001" />
 	    </inertial>
 	    <visual>
@@ -16,9 +16,7 @@
 	    </visual>
 	    <collision>
-		<laser_retro>0</laser_retro>
-		<max_contacts>10</max_contacts>
 		<origin xyz="0.0 0.0 0.0" rpy="0 0 0" />
 		<geometry>
-		    <box size="0.005 0.03 0.03" />
+		    <box size="0.03 0.16 0.03" />
 		</geometry>
 	    </collision>
@@ -32,18 +30,18 @@
 		        <update_rate>30.0</update_rate>
 		        <camera name="head">
-		            <horizontal_fov>1.085594795</horizontal_fov>
+		            <horizontal_fov>1.3962634</horizontal_fov>
 		            <image>
-		                <width>640</width>
-		                <height>480</height>
+		                <width>1280</width>
+		                <height>720</height>
 		                <format>R8G8B8</format>
 		            </image>
 		            <clip>
 		                <near>0.02</near>
-		                <far>100</far>
+		                <far>300</far>
 		            </clip>
 		            <noise>
 		                <type>gaussian</type>
 		                <mean>0.0</mean>
-		                <stddev>0.0</stddev>
+		                <stddev>0.007</stddev>
 		            </noise>
 		        </camera>

File: racecar_description/urdf/sensors/lidar.xacro (robot description, xacro)
@@ -36,13 +36,13 @@
                     <scan>
                         <horizontal>
-                            <samples>1081</samples>
+                            <samples>360</samples>
                             <resolution>1</resolution>
-                            <min_angle>-2.3561944902</min_angle>
-                            <max_angle>2.3561944902</max_angle>
+                            <min_angle>-3.1415926</min_angle>
+                            <max_angle>3.1415926</max_angle>
                         </horizontal>
                     </scan>
                     <range>
                         <min>0.10</min>
-                        <max>30.0</max>
+                        <max>8.0</max>
                         <resolution>0.01</resolution>
                     </range>
